File: eZ-E36-brakeout/eZ-E36-brakeout.kicad_pcb (KiCad board)
At the start: 2 copper layers, 88.9 x 40.6 mm, 12 parts, among them J1 Conn_02x13_Top_Bottom, J11 Conn_01x13_Pin, J12 Conn_01x13_Pin, J2 Conn_02x13_Top_Bottom, J21 Conn_01x13_Pin, J22 Conn_01x13_Pin, J3 Conn_02x06_Top_Bottom, J31 Conn_01x06_Pin, J32 Conn_01x06_Pin, J4 Conn_01x06_Pin, J41 Conn_01x06_Pin

Commit message: Reorganize and update project with recent work.
Other:
- board text added: "X16 White"
- board text added: "X17 Blue"
- board text added: "eZ E36 Cluster Breakout By: Luca van Straaten Version 1.1"
